File: usb-pd.kicad_sch (KiCad schematic)
At the start: 66 parts, among them J3 USB-C_GCT_USB4105-GF-A, Q4 BSS138-7-F, Q6 SQS401EN-T1_BE3, Q8 BSS138-7-F, Q9 BSS138-7-F, U5 CYPD3177-24LQXQ, U9 SIC477ED-T1-GE3

Commit message: [#79262] DRC clean
Changed lines of the file:
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@@
 	)
 	(junction
+		(at 331.47 194.31)
+		(diameter 0)
+		(color 0 0 0 0)
+	)
+	(junction
 		(at 269.24 53.34)
 		(diameter 0)
@@
 	(wire
 		(pts
-			(xy 323.85 194.31) (xy 328.93 194.31)
+			(xy 323.85 194.31) (xy 331.47 194.31)
 		)
 		(stroke
@@
 	(wire
 		(pts
+			(xy 331.47 191.77) (xy 331.47 194.31)
+		)
+		(stroke
+			(width 0)
+			(type default)
+		)
+	)
+	(wire
+		(pts
 			(xy 172.72 53.34) (xy 172.72 73.66)
 		)
@@
 	(wire
 		(pts
+			(xy 331.47 194.31) (xy 334.01 194.31)
+		)
+		(stroke
+			(width 0)
+			(type default)
+		)
+	)
+	(wire
+		(pts
 			(xy 133.35 220.98) (xy 176.53 220.98)
 		)
@@
 	)
 	(table
+		(column_count 1)
+		(border
+			(external yes)
+			(header yes)
+			(stroke
+				(width 0)
+				(type solid)
+			)
+		)
+		(separators
+			(rows yes)
+			(cols yes)
+			(stroke
+				(width 0)
+				(type solid)
+			)
+		)
+		(column_widths 69.85)
+		(row_heights 3.81)
+		(cells
+			(table_cell "CONFIGURATION"
+				(exclude_from_sim no)
+				(at 330.2 26.67 0)
+				(size 69.85 3.81)
+				(margins 0.9525 0.9525 0.9525 0.9525)
+				(span 1 1)
+				(fill
+					(type none)
+				)
+				(effects
+					(font
+						(size 1.27 1.27)
+					)
+					(justify left top)
+				)
+			)
+		)
+	)
+	(table
 		(column_count 2)
 		(border
@@
 		)
 	)
-	(table
-		(column_count 1)
-		(border
-			(external yes)
-			(header yes)
-			(stroke
-				(width 0)
-				(type solid)
-			)
-		)
-		(separators
-			(rows yes)
-			(cols yes)
-			(stroke
-				(width 0)
-				(type solid)
-			)
-		)
-		(column_widths 69.85)
-		(row_heights 3.81)
-		(cells
-			(table_cell "CONFIGURATION"
-				(exclude_from_sim no)
-				(at 330.2 26.67 0)
-				(size 69.85 3.81)
-				(margins 0.9525 0.9525 0.9525 0.9525)
-				(span 1 1)
-				(fill
-					(type none)
-				)
-				(effects
-					(font
-						(size 1.27 1.27)
-					)
-					(justify left top)
-				)
-			)
-		)
-	)
 	(label "VDDD_3V3"
 		(at 332.74 50.8 0)
@@
 	(hierarchical_label "12V_OUT"
 		(shape output)
-		(at 328.93 194.31 0)
+		(at 334.01 194.31 0)
 		(effects
 			(font
@@
 					(unit 1)
 				)
+			)
+		)
+	)
+	(symbol
+		(lib_id "antmicropower:PWR_FLAG")
+		(at 331.47 191.77 0)
+		(unit 1)
+		(exclude_from_sim no)
+		(in_bom yes)
+		(on_board yes)
+		(dnp no)
+		(property "Reference" "#FLG04"
+			(at 331.47 189.865 0)
+			(effects
+				(font
+					(size 1.27 1.27)
+				)
+				(hide yes)
+			)
+		)
+		(property "Value" "PWR_FLAG"
+			(at 337.82 189.865 0)
+			(effects
+				(font
+					(size 1.27 1.27)
+				)
+			)
+		)
+		(property "Footprint" ""
+			(at 331.47 191.77 0)
+			(effects
+				(font
+					(size 1.27 1.27)
+				)
+				(hide yes)
+			)
+		)
+		(property "Datasheet" ""
+			(at 331.47 191.77 0)
+			(effects
+				(font
+					(size 1.27 1.27)
+				)
+				(hide yes)
+			)
+		)
+		(property "Description" ""
+			(at 331.47 191.77 0)
+			(effects
+				(font
+					(size 1.27 1.27)
+				)
+				(hide yes)
+			)
+		)
+		(pin "1"
+		)
+		(instances
+			(project "oculink-to-pcie-adapter"
+				(path "/44c3be85-0a18-4d93-a9a5-650ee09b6032/967dc2ce-6faa-4f65-adf2-eb5d333aef74"
+					(reference "#FLG04")
+					(unit 1)
+				)
