File: pcie-clock-generator.kicad_sch (KiCad schematic)
At the start: 7 parts, among them U31 SI52112-B6-GT, Y6 Resonator_25MHz_ABM8G

Commit message: [#79262] WIP: Component placement
Connections:
- net at C133.2, Y6.1: now also U31.3 (XIN/CLKIN); no longer U31.2 (XOUT)
- net at C134.2, Y6.3: now also U31.2 (XOUT); no longer U31.3 (XIN/CLKIN)
Other:
- moved on the sheet: C133, C134
